Commit message: before format

File: src/install/manipulator_description/share/manipulator_description/urdf/manipulator.urdf.xacro (robot description, xacro)
@@ -236,12 +236,6 @@
             <plugin filename="gz-sim-sensors-system" name="gz::sim::systems::Sensors">
                 <render_engine>ogre2</render_engine>
-            </plugin>
-        </xacro:unless>
-        <plugin filename="gz-sim-mimic-joint-system" name="gz::sim::systems::MimicJoint">
-            <joint>joint_4</joint>
-            <mimic_joint>joint_5</mimic_joint>
-            <multiplier>-1.0</multiplier>
-            <offset>0.0</offset>
         </plugin>
+      </xacro:unless>
     </gazebo>
 </robot>

File: src/install/manipulator_description/share/manipulator_description/urdf/manipulator_ros2_control.xacro (robot description, xacro)
@@ -1,8 +1,6 @@
 <?xml version="1.0"?>
-<robot xmlns:xacro="http://www.ros.org/wiki/xacro" name="arduinobot">
-    <ros2_control name="RobotSystem" type="system">
-        <xacro:property name="PI" value="3.14159265359" />
-        <!-- ros2_control Gazebo -->
-        <!-- ROS 2 Humble -->
+<robot xmlns:xacro="http://www.ros.org/wiki/xacro" name="manipulator">
+    <xacro:property name="PI" value="3.14159265359" />
+    <ros2_control type="system" name="robot_system">
         <xacro:if value="$(arg is_ignition)">
             <hardware>
@@ -10,5 +8,4 @@
             </hardware>
         </xacro:if>
-        <!-- ROS 2 Iron or above -->
         <xacro:unless value="$(arg is_ignition)">
             <hardware>
@@ -18,6 +15,6 @@
         <joint name="joint_1">
             <command_interface name="position">
-            <param name="min">-${PI / 2}</param>
-            <param name="max">${PI / 2}</param>
+               <param name="min">-${PI / 2}</param>
+               <param name="max">${PI / 2}</param>
             </command_interface>
             <state_interface name="position"/>
@@ -25,6 +22,6 @@
         <joint name="joint_2">
             <command_interface name="position">
-            <param name="min">-${PI / 2}</param>
-            <param name="max">${PI / 2}</param>
+               <param name="min">-${PI / 2}</param>
+               <param name="max">${PI / 2}</param>
             </command_interface>
             <state_interface name="position"/>
@@ -32,6 +29,6 @@
         <joint name="joint_3">
             <command_interface name="position">
-            <param name="min">-${PI / 2}</param>
-            <param name="max">${PI / 2}</param>
+               <param name="min">-${PI / 2}</param>
+               <param name="max">${PI / 2}</param>
             </command_interface>
             <state_interface name="position"/>
@@ -39,6 +36,6 @@
         <joint name="joint_4">
             <command_interface name="position">
-            <param name="min">-${PI / 2}</param>
-            <param name="max">0.0</param>
+               <param name="min">-${PI / 2}</param>
+               <param name="max">0.0</param>
             </command_interface>
             <state_interface name="position"/>
@@ -47,4 +44,5 @@
             <param name="mimic">joint_4</param>
             <param name="multiplier">-1</param>
+            <state_interface name="position"/>
         </joint>
     </ros2_control>
