Commit message: initial

File: install/manipulator_description/share/manipulator_description/urdf/manipulator.urdf.xacro (robot description, xacro)
@@ -224,5 +224,5 @@
         <xacro:if value="$(arg is_ignition)">
             <plugin filename="ign_ros2_control-system" name="ign_ros2_control::IgnitionROS2ControlPlugin">
-                <parameters>$(find manipulator_description)/config/manipulator_controllers.yaml</parameters>
+                <parameters>$(find manipulator_controller)/config/manipulator_controller.yaml</parameters>
             </plugin>
             <plugin filename="ignition-gazebo-sensors-system" name="ignition::gazebo::systems::Sensors">
@@ -232,10 +232,16 @@
         <xacro:unless value="$(arg is_ignition)">
             <plugin filename="gz_ros2_control-system" name="gz_ros2_control::GazeboSimROS2ControlPlugin">
-                <parameters>$(find manipulator_description)/config/manipulator_controllers.yaml</parameters>
+                <parameters>$(find manipulator_controller)/config/manipulator_controller.yaml</parameters>
             </plugin>
             <plugin filename="gz-sim-sensors-system" name="gz::sim::systems::Sensors">
                 <render_engine>ogre2</render_engine>
+            </plugin>
+        </xacro:unless>
+        <plugin filename="gz-sim-mimic-joint-system" name="gz::sim::systems::MimicJoint">
+            <joint>joint_4</joint>
+            <mimic_joint>joint_5</mimic_joint>
+            <multiplier>-1.0</multiplier>
+            <offset>0.0</offset>
         </plugin>
-      </xacro:unless>
     </gazebo>
 </robot>

File: install/manipulator_description/share/manipulator_description/urdf/manipulator_ros2_control.xacro (robot description, xacro)
@@ -1,11 +1,14 @@
 <?xml version="1.0"?>
-<robot xmlns:xacro="http://www.ros.org/wiki/xacro" name="manipulator">
-    <xacro:property name="PI" value="3.14159265359" />
-    <ros2_control type="system" name="robot_system">
+<robot xmlns:xacro="http://www.ros.org/wiki/xacro" name="arduinobot">
+    <ros2_control name="RobotSystem" type="system">
+        <xacro:property name="PI" value="3.14159265359" />
+        <!-- ros2_control Gazebo -->
+        <!-- ROS 2 Humble -->
         <xacro:if value="$(arg is_ignition)">
             <hardware>
-                <plugin>ign_ros2_control/IgnitionSystemPlugin</plugin>
+                <plugin>ign_ros2_control/IgnitionSystem</plugin>
             </hardware>
         </xacro:if>
+        <!-- ROS 2 Iron or above -->
         <xacro:unless value="$(arg is_ignition)">
             <hardware>
@@ -15,6 +18,6 @@
         <joint name="joint_1">
             <command_interface name="position">
-               <param name="min">-${PI / 2}</param>
-               <param name="max">${PI / 2}</param>
+            <param name="min">-${PI / 2}</param>
+            <param name="max">${PI / 2}</param>
             </command_interface>
             <state_interface name="position"/>
@@ -22,6 +25,6 @@
         <joint name="joint_2">
             <command_interface name="position">
-               <param name="min">-${PI / 2}</param>
-               <param name="max">${PI / 2}</param>
+            <param name="min">-${PI / 2}</param>
+            <param name="max">${PI / 2}</param>
             </command_interface>
             <state_interface name="position"/>
@@ -29,6 +32,6 @@
         <joint name="joint_3">
             <command_interface name="position">
-               <param name="min">-${PI / 2}</param>
-               <param name="max">${PI / 2}</param>
+            <param name="min">-${PI / 2}</param>
+            <param name="max">${PI / 2}</param>
             </command_interface>
             <state_interface name="position"/>
@@ -36,6 +39,6 @@
         <joint name="joint_4">
             <command_interface name="position">
-               <param name="min">-${PI / 2}</param>
-               <param name="max">0.0</param>
+            <param name="min">-${PI / 2}</param>
+            <param name="max">0.0</param>
             </command_interface>
             <state_interface name="position"/>

File: install/manipulator_description/share/manipulator_description/urdf/manupilator_gazebo.xacro (robot description, xacro)
@@ -4,10 +4,10 @@
         <xacro:if value="$(arg is_ignition)">
             <plugin filename="ign_ros2_control-system" name="ign_ros2_control::IgnitionROS2ControlPlugin">
-                <parameters></parameters>
+                <parameters>$(find manipulator_controller)/config/manipulator_controller.yaml</parameters>
             </plugin>
         </xacro:if>
         <xacro:unless value="$(arg is_ignition)">
             <plugin filename="gz_ros2_control-system" name="gz_ros2_control::GazeboSimROS2ControlPlugin">
-                <parameters></parameters>
+                <parameters>$(find manipulator_controller)/config/manipulator_controller.yaml</parameters>
             </plugin>
         </xacro:unless>

File: src/manipulator_description/urdf/manipulator.urdf.xacro (robot description, xacro)
@@ -1,124 +1,138 @@
 <?xml version="1.0"?>
 <robot xmlns:xacro="http://www.ros.org/wiki/xacro" name="manipulator">
-    <xacro:arg name="is_ignition" default="true"/>
-    <xacro:include filename="$(find manipulator_description)/urdf/manupilator_gazebo.xacro"/>
-    <xacro:include filename="$(find manipulator_description)/urdf/manipulator_ros2_control.xacro"/>
+    <xacro:arg name="is_ignition" default="true" />
+    <xacro:include filename="$(find manipulator_description)/urdf/manupilator_gazebo.xacro" />
+    <xacro:include filename="$(find manipulator_description)/urdf/manipulator_ros2_control.xacro" />
     <!-- Useful XACRO Variables (Properties) -->
     <xacro:property name="PI" value="3.14159265359" />
     <xacro:property name="effort" value="30.0" />
     <xacro:property name="velocity" value="10.0" />
-    <xacro:arg name="is_ignition" default="true"/>
+    <xacro:arg name="is_ignition" default="true" />
     <xacro:macro name="default_inertial" params="mass">
         <inertial>
             <mass value="${mass}" />
             <inertia ixx="1.0" ixy="0.0" ixz="0.0"
-                     iyy="1.0" iyz="0.0"
-                     izz="1.0" />
+                iyy="1.0" iyz="0.0"
+                izz="1.0" />
         </inertial>
     </xacro:macro>
     <!-- Links -->
-    <link name="world"/>
+    <link name="world" />
     <link name="base_link">
-        <xacro:default_inertial mass="1.0"/>
-        <visual>
-            <origin rpy="0 0 0" xyz="-0.5 -0.5 0"/>
-            <geometry>
-                <mesh filename="package://manipulator_description/meshes/basement.STL" scale="0.01 0.01 0.01"/>
-            </geometry>
-        </visual>
-        <collision>
-            <origin rpy="0 0 0" xyz="-0.5 -0.5 0"/>
-            <geometry>
-                <mesh filename="package://manipulator_description/meshes/basement.STL" scale="0.01 0.01 0.01"/>
+        <xacro:default_inertial mass="1.0" />
+        <visual>
+            <origin rpy="0 0 0" xyz="-0.5 -0.5 0" />
+            <geometry>
+                <mesh filename="package://manipulator_description/meshes/basement.STL"
+                    scale="0.01 0.01 0.01" />
+            </geometry>
+        </visual>
+        <collision>
+            <origin rpy="0 0 0" xyz="-0.5 -0.5 0" />
+            <geometry>
+                <mesh filename="package://manipulator_description/meshes/basement.STL"
+                    scale="0.01 0.01 0.01" />
             </geometry>
         </collision>
     </link>
     <link name="base_plate">
-        <xacro:default_inertial mass="0.1"/>
-        <visual>
-            <origin rpy="0 0 0" xyz="-0.39 -0.39 -0.56"/>
-            <geometry>
-                <mesh filename="package://manipulator_description/meshes/base_plate.STL" scale="0.01 0.01 0.01"/>
-            </geometry>
-        </visual>
-        <collision>
-            <origin rpy="0 0 0" xyz="-0.39 -0.39 -0.56"/>
-            <geometry>
-                <mesh filename="package://manipulator_description/meshes/base_plate.STL" scale="0.01 0.01 0.01"/>
+        <xacro:default_inertial mass="0.1" />
+        <visual>
+            <origin rpy="0 0 0" xyz="-0.39 -0.39 -0.56" />
+            <geometry>
+                <mesh filename="package://manipulator_description/meshes/base_plate.STL"
+                    scale="0.01 0.01 0.01" />
+            </geometry>
+        </visual>
+        <collision>
+            <origin rpy="0 0 0" xyz="-0.39 -0.39 -0.56" />
+            <geometry>
+                <mesh filename="package://manipulator_description/meshes/base_plate.STL"
+                    scale="0.01 0.01 0.01" />
             </geometry>
         </collision>
     </link>
     <link name="forward_drive_arm">
-        <xacro:default_inertial mass="0.1"/>
-        <visual>
-            <origin rpy=" 0 -${PI / 2} ${PI / 2}" xyz="0.19 0.06 -0.08"/>
-            <geometry>
-                <mesh filename="package://manipulator_description/meshes/forward_drive_arm.STL" scale="0.01 0.01 0.01"/>
-            </geometry>
-        </visual>
-        <collision>
-            <origin rpy=" 0 -${PI / 2} ${PI / 2}" xyz="0.19 0.06 -0.08"/>
-            <geometry>
-                <mesh filename="package://manipulator_description/meshes/forward_drive_arm.STL" scale="0.01 0.01 0.01"/>
+        <xacro:default_inertial mass="0.1" />
+        <visual>
+            <origin rpy=" 0 -${PI / 2} ${PI / 2}" xyz="0.19 0.06 -0.08" />
+            <geometry>
+                <mesh filename="package://manipulator_description/meshes/forward_drive_arm.STL"
+                    scale="0.01 0.01 0.01" />
+            </geometry>
+        </visual>
+        <collision>
+            <origin rpy=" 0 -${PI / 2} ${PI / 2}" xyz="0.19 0.06 -0.08" />
+            <geometry>
+                <mesh filename="package://manipulator_description/meshes/forward_drive_arm.STL"
+                    scale="0.01 0.01 0.01" />
             </geometry>
         </collision>
     </link>
     <link name="horizontal_arm">
-        <xacro:default_inertial mass="0.1"/>
-        <visual>
-            <origin rpy="${PI / 2} 0 ${PI / 2}" xyz="-0.03 -0.4 -0.06"/>
-            <geometry>
-                <mesh filename="package://manipulator_description/meshes/horizontal_arm.STL" scale="0.01 0.01 0.01"/>
-            </geometry>
-        </visual>
-        <collision>
-            <origin rpy="${PI / 2} 0 ${PI / 2}" xyz="-0.03 -0.4 -0.06"/>
-            <geometry>
-                <mesh filename="package://manipulator_description/meshes/horizontal_arm.STL" scale="0.01 0.01 0.01"/>
+        <xacro:default_inertial mass="0.1" />
+        <visual>
+            <origin rpy="${PI / 2} 0 ${PI / 2}" xyz="-0.03 -0.4 -0.06" />
+            <geometry>
+                <mesh filename="package://manipulator_description/meshes/horizontal_arm.STL"
+                    scale="0.01 0.01 0.01" />
+            </geometry>
+        </visual>
+        <collision>
+            <origin rpy="${PI / 2} 0 ${PI / 2}" xyz="-0.03 -0.4 -0.06" />
+            <geometry>
+                <mesh filename="package://manipulator_description/meshes/horizontal_arm.STL"
+                    scale="0.01 0.01 0.01" />
             </geometry>
         </collision>
     </link>
     <link name="claw_support">
-        <xacro:default_inertial mass="0.05"/>
-        <visual>
-            <origin rpy="0 0 ${PI / 2}" xyz="0 -0.05 -0.15"/>
-            <geometry>
-                <mesh filename="package://manipulator_description/meshes/claw_support.STL" scale="0.01 0.01 0.01"/>
-            </geometry>
-        </visual>
-        <collision>
-            <origin rpy="0 0 ${PI / 2}" xyz="0 -0.05 -0.15"/>
-            <geometry>
-                <mesh filename="package://manipulator_description/meshes/claw_support.STL" scale="0.01 0.01 0.01"/>
+        <xacro:default_inertial mass="0.05" />
+        <visual>
+            <origin rpy="0 0 ${PI / 2}" xyz="0 -0.05 -0.15" />
+            <geometry>
+                <mesh filename="package://manipulator_description/meshes/claw_support.STL"
+                    scale="0.01 0.01 0.01" />
+            </geometry>
+        </visual>
+        <collision>
+            <origin rpy="0 0 ${PI / 2}" xyz="0 -0.05 -0.15" />
+            <geometry>
+                <mesh filename="package://manipulator_description/meshes/claw_support.STL"
+                    scale="0.01 0.01 0.01" />
             </geometry>
         </collision>
     </link>
     <link name="gripper_right">
-        <xacro:default_inertial mass="0.01"/>
-        <visual>
-            <origin rpy="0 0 -${PI / 2}" xyz="-0.1 0.50 -0.1"/>
-            <geometry>
-                <mesh filename="package://manipulator_description/meshes/right_finger.STL" scale="0.01 0.01 0.01"/>
-            </geometry>
-        </visual>
-        <collision>
-            <origin rpy="0 0 -${PI / 2}" xyz="-0.1 0.50 -0.1"/>
-            <geometry>
-                <mesh filename="package://manipulator_description/meshes/right_finger.STL" scale="0.01 0.01 0.01"/>
+        <xacro:default_inertial mass="0.01" />
+        <visual>
+            <origin rpy="0 0 -${PI / 2}" xyz="-0.1 0.50 -0.1" />
+            <geometry>
+                <mesh filename="package://manipulator_description/meshes/right_finger.STL"
+                    scale="0.01 0.01 0.01" />
+            </geometry>
+        </visual>
+        <collision>
+            <origin rpy="0 0 -${PI / 2}" xyz="-0.1 0.50 -0.1" />
+            <geometry>
+                <mesh filename="package://manipulator_description/meshes/right_finger.STL"
+                    scale="0.01 0.01 0.01" />
             </geometry>
         </collision>
     </link>
     <link name="gripper_left">
-        <xacro:default_inertial mass="0.01"/>
-        <visual>
-            <origin rpy="0 0 -${PI / 2}" xyz="-0.04 0.50 -0.1"/>
-            <geometry>
-                <mesh filename="package://manipulator_description/meshes/left_finger.STL" scale="0.01 0.01 0.01"/>
-            </geometry>
-        </visual>
-        <collision>
-            <origin rpy="0 0 -${PI / 2}" xyz="-0.04 0.50 -0.1"/>
-            <geometry>
-                <mesh filename="package://manipulator_description/meshes/left_finger.STL" scale="0.01 0.01 0.01"/>
+        <xacro:default_inertial mass="0.01" />
+        <visual>
+            <origin rpy="0 0 -${PI / 2}" xyz="-0.04 0.50 -0.1" />
+            <geometry>
+                <mesh filename="package://manipulator_description/meshes/left_finger.STL"
+                    scale="0.01 0.01 0.01" />
+            </geometry>
+        </visual>
+        <collision>
+            <origin rpy="0 0 -${PI / 2}" xyz="-0.04 0.50 -0.1" />
+            <geometry>
+                <mesh filename="package://manipulator_description/meshes/left_finger.STL"
+                    scale="0.01 0.01 0.01" />
             </geometry>
         </collision>
@@ -150,15 +164,17 @@
     </gazebo>
     <link name="rgb_camera">
-        <xacro:default_inertial mass="0.001"/>
-        <visual>
-            <origin rpy="-1.57 0 -1.57" xyz="-0.1 0.125 0.15"/>
-            <geometry>
-                <mesh filename="package://manipulator_description/meshes/pi_camera.STL" scale="0.01 0.01 0.01"/>
-            </geometry>
-        </visual>
-        <collision>
-            <origin rpy="-1.57 0 -1.57" xyz="-0.1 0.125 0.15"/>
-            <geometry>
-                <mesh filename="package://manipulator_description/meshes/pi_camera.STL" scale="0.01 0.01 0.01"/>
+        <xacro:default_inertial mass="0.001" />
+        <visual>
+            <origin rpy="-1.57 0 -1.57" xyz="-0.1 0.125 0.15" />
+            <geometry>
+                <mesh filename="package://manipulator_description/meshes/pi_camera.STL"
+                    scale="0.01 0.01 0.01" />
+            </geometry>
+        </visual>
+        <collision>
+            <origin rpy="-1.57 0 -1.57" xyz="-0.1 0.125 0.15" />
+            <geometry>
+                <mesh filename="package://manipulator_description/meshes/pi_camera.STL"
+                    scale="0.01 0.01 0.01" />
             </geometry>
         </collision>
@@ -166,70 +182,73 @@
     <!-- Joints -->
     <joint name="virtual_joint" type="fixed">
-        <parent link="world"/>
-        <child link="base_link"/>
-        <origin xyz="0 0 0" rpy="0 0 0"/>
-    </joint>
-    <joint name ="joint_1" type="revolute">
-        <parent link="base_link"/>
-        <child link = "base_plate"/>
-        <origin xyz="0 0 0.307"/>
-        <axis xyz="0 0 1"/>
+        <parent link="world" />
+        <child link="base_link" />
+        <origin xyz="0 0 0" rpy="0 0 0" />
+    </joint>
+    <joint name="joint_1" type="revolute">
+        <parent link="base_link" />
+        <child link="base_plate" />
+        <origin xyz="0 0 0.307" />
+        <axis xyz="0 0 1" />
         <limit lower="-${PI / 2}" upper="${PI / 2}"
-               effort="${effort}" velocity="${velocity}"/>
-    </joint>
-    <joint name ="joint_2" type="revolute">
-        <parent link="base_plate"/>
-        <child link = "forward_drive_arm"/>
-        <origin xyz="-0.02 0 0.35"/>
-        <axis xyz="1 0 0"/>
+            effort="${effort}" velocity="${velocity}" />
+    </joint>
+    <joint name="joint_2" type="revolute">
+        <parent link="base_plate" />
+        <child link="forward_drive_arm" />
+        <origin xyz="-0.02 0 0.35" />
+        <axis xyz="1 0 0" />
         <limit lower="-${PI / 2}" upper="${PI / 2}"
-                effort="${effort}" velocity="${velocity}"/>
-    </joint>
-    <joint name ="joint_3" type="revolute">
-        <parent link="forward_drive_arm"/>
-        <child link = "horizontal_arm"/>
-        <origin xyz="0 0 0.8"/>
-        <axis xyz="1 0 0"/>
+            effort="${effort}" velocity="${velocity}" />
+    </joint>
+    <joint name="joint_3" type="revolute">
+        <parent link="forward_drive_arm" />
+        <child link="horizontal_arm" />
+        <origin xyz="0 0 0.8" />
+        <axis xyz="1 0 0" />
         <limit lower="-${PI / 2}" upper="${PI / 2}"
-               effort="${effort}" velocity="${velocity}"/>
-    </joint>
-    <joint name ="horizontal_arm_to_claw_support" type="fixed">
-        <parent link="horizontal_arm"/>
-        <child link = "claw_support"/>
-        <origin xyz="0 0.82 0"/>
-    </joint>
-    <joint name ="joint_4" type="revolute">
-        <parent link="claw_support"/>
-        <child link = "gripper_right"/>
-        <origin xyz="-0.04 0.13 -0.1"/>
-        <axis xyz="0 0 1"/>
+            effort="${effort}" velocity="${velocity}" />
+    </joint>
+    <joint name="horizontal_arm_to_claw_support" type="fixed">
+        <parent link="horizontal_arm" />
+        <child link="claw_support" />
+        <origin xyz="0 0.82 0" />
+    </joint>
+    <joint name="joint_4" type="revolute">
+        <parent link="claw_support" />
+        <child link="gripper_right" />
+        <origin xyz="-0.04 0.13 -0.1" />
+        <axis xyz="0 0 1" />
         <limit lower="-${PI / 2}" upper="0.0"
-               effort="${effort}" velocity="${velocity}"/>
-    </joint>
-    <joint name ="joint_5" type="revolute">
-        <parent link="claw_support"/>
-        <child link = "gripper_left"/>
-        <origin xyz="-0.22 0.13 -0.1"/>
-        <axis xyz="0 0 1"/>
+            effort="${effort}" velocity="${velocity}" />
+    </joint>
+    <joint name="joint_5" type="revolute">
+        <parent link="claw_support" />
+        <child link="gripper_left" />
+        <origin xyz="-0.22 0.13 -0.1" />
+        <axis xyz="0 0 1" />
         <limit lower="0.0" upper="${PI / 2}"
-               effort="${effort}" velocity="${velocity}"/>
-        <mimic joint="joint_4" multiplier="-1"/>
-    </joint>
-    <joint name ="rgb_camera_joint" type="fixed">
-        <parent link="base_link"/>
-        <child link = "rgb_camera"/>
-        <origin rpy="0 -0.5 1.57" xyz="0 0.45 0.2"/>
+            effort="${effort}" velocity="${velocity}" />
+        <mimic joint="joint_4" multiplier="-1" />
+    </joint>
+    <joint name="rgb_camera_joint" type="fixed">
+        <parent link="base_link" />
+        <child link="rgb_camera" />
+        <origin rpy="0 -0.5 1.57" xyz="0 0.45 0.2" />
     </joint>
     <gazebo>
         <xacro:if value="$(arg is_ignition)">
-            <plugin filename="ign_ros2_control-system" name="ign_ros2_control::IgnitionROS2ControlPlugin">
+            <plugin filename="ign_ros2_control-system"
+                name="ign_ros2_control::IgnitionROS2ControlPlugin">
                 <parameters>$(find manipulator_controller)/config/manipulator_controller.yaml</parameters>
             </plugin>
-            <plugin filename="ignition-gazebo-sensors-system" name="ignition::gazebo::systems::Sensors">
+            <plugin filename="ignition-gazebo-sensors-system"
+                name="ignition::gazebo::systems::Sensors">
                 <render_engine>ogre2</render_engine>
             </plugin>
         </xacro:if>
         <xacro:unless value="$(arg is_ignition)">
-            <plugin filename="gz_ros2_control-system" name="gz_ros2_control::GazeboSimROS2ControlPlugin">
+            <plugin filename="gz_ros2_control-system"
+                name="gz_ros2_control::GazeboSimROS2ControlPlugin">
                 <parameters>$(find manipulator_controller)/config/manipulator_controller.yaml</parameters>
             </plugin>
@@ -238,10 +257,4 @@
             </plugin>
         </xacro:unless>
-        <plugin filename="gz-sim-mimic-joint-system" name="gz::sim::systems::MimicJoint">
-            <joint>joint_4</joint>
-            <mimic_joint>joint_5</mimic_joint>
-            <multiplier>-1.0</multiplier>
-            <offset>0.0</offset>
-        </plugin>
     </gazebo>
 </robot>
